Commit message: 10 enero

File: Versions/Actual_version/boat_subdivided4.xacro (robot description, xacro)
@@ -11,6 +11,6 @@
     <xacro:property name="middle_water_displaced_mass" value="40"/>
     <xacro:property name="front_water_displaced_mass" value="25"/>
-    <xacro:property name="scalex" value=".19"/>
-    <xacro:property name="scaley" value=".085"/>
+    <xacro:property name="scalex" value=".193"/>
+    <xacro:property name="scaley" value=".117"/>
     <xacro:property name="scalez" value=".1"/>
     <xacro:property name="bl1" value=".1" />
@@ -356,13 +356,13 @@
             <collision name="collision">
                 <geometry>
-                  <box size="${0.2*scalex} ${0.02*scaley} ${0.3*scalez}" />
+                  <box size="${0.05} ${0.005} ${0.142}" />
                 </geometry>
-                <origin rpy="0 0 0" xyz="${-0.1*scalex} 0 0"/>
+                <origin rpy="0 0 0" xyz="0 0 0"/>
             </collision>
             <visual name="visual">
                 <geometry>
-                  <mesh filename="package://usv_sim/meshes/simpleHull3/box.dae" scale="${0.2*scalex} ${0.02*scaley} ${0.3*scalez}"/>
+                  <mesh filename="package://usv_sim/meshes/simpleHull3/box.dae" scale="${0.05} ${0.005} ${0.142}"/>
                 </geometry>
-                <origin rpy="0 0 0" xyz="${-0.1*scalex} 0 0"/>
+                <origin rpy="0 0 0" xyz="0 0 0"/>
             </visual>
         </link>
@@ -370,5 +370,5 @@
             <parent link="back_r_link"/>
             <child link="rudder"/>
-            <origin rpy="0 0 0" xyz="${-1.4*scalex} ${0.39*scaley} ${-0.5*scalez}"/>
+            <origin rpy="0 0 0" xyz="-0.2 0 -0.12"/>
             <dynamics damping="1.0"/>
             <axis xyz="0 0 1"/>
@@ -386,13 +386,13 @@
     <link name="hokuyo_link">
         <collision name="collision">
-	        <origin xyz="0 0 0" rpy="0 0 0"/>
+	        <origin xyz="-0.45 0 -0.15" rpy="0 0 0"/>
 	        <geometry>
-	        	<box size="0.1 0.1 0.1"/>
+	        	<box size="0.05 0.05 0.05"/>
 	        </geometry>
         </collision>
         <visual name="visual">
-        	<origin xyz="0 0 0" rpy="0 0 0"/>
+        	<origin xyz="-0.45 0 -0.15" rpy="0 0 0"/>
         	<geometry>
-        		<mesh filename="package://usv_sim/meshes/simpleHull3/box.dae" scale="0.1 0.1 0.1"/>
+        		<mesh filename="package://usv_sim/meshes/simpleHull3/box.dae" scale="0.05 0.05 0.05"/>
         	</geometry>
         </visual>

File: Versions/Actual_version/sailboat.xacro (robot description, xacro)
@@ -11,5 +11,5 @@
     <xacro:property name="scale_V2Y" value="0.335"/>
     <xacro:property name="scale_V2Z" value="0.51"/>
-    <xacro:property name="Angle_Sail2" value="3"/>
+    <xacro:property name="Angle_Sail2" value="3.14"/>
     <xacro:property name="SailXo" value="0"/>
     <xacro:property name="SailYo" value="0"/>
@@ -118,5 +118,5 @@
         <parent link="base_link"/>
         <child link="keel"/>
-        <origin rpy="0 0 0" xyz="0 0 -0.35"/>
+        <origin rpy="0 0 0" xyz="0 0 -0.12"/>
         <dynamics damping="1.0"/>
         <axis xyz="0 0 1"/>

Commit message: 21 feb

File: Versions/Actual_version/boat_subdivided4.xacro (robot description, xacro)
@@ -5,7 +5,7 @@
     <xacro:property name="front_body_mass" value="5"/>
     <xacro:property name="back_body_mass" value="5"/>
-    <xacro:property name="middle_body_mass" value="5"/>
-    <xacro:property name="rear_body_mass" value="5"/>
-    <xacro:property name="front_body_mass" value="2"/>
+    <xacro:property name="middle_body_mass" value="0.2"/>
+    <xacro:property name="rear_body_mass" value="0.2"/>
+    <xacro:property name="front_body_mass" value="0.2"/>
     <xacro:property name="back_water_displaced_mass" value="40"/>
     <xacro:property name="middle_water_displaced_mass" value="40"/>
@@ -345,5 +345,5 @@
         <link name="rudder">
             <inertial>
-                <mass value="1" />
+                <mass value="0.2" />
                 <inertia
                   ixx="0.05"
@@ -370,5 +370,5 @@
             <parent link="back_r_link"/>
             <child link="rudder"/>
-            <origin rpy="0 0 0" xyz="-0.2 0 -0.12"/>
+            <origin rpy="0 0 0" xyz="-0.2 0 -0.10"/>
             <dynamics damping="1.0"/>
             <axis xyz="0 0 1"/>

File: Versions/Actual_version/sailboat.xacro (robot description, xacro)
@@ -12,5 +12,5 @@
     <xacro:property name="scale_V2Z" value="0.51"/>
     <xacro:property name="Angle_Sail2" value="3.14"/>
-    <xacro:property name="SailXo" value="0"/>
+    <xacro:property name="SailXo" value="0.04"/>
     <xacro:property name="SailYo" value="0"/>
     <xacro:property name="SailZo" value="-0.041"/>
@@ -23,5 +23,5 @@
 		<inertial>
 		    	<origin rpy="0 0 0" xyz="-0.3 0 0.4"/>
-			<mass value="1" />
+			<mass value="0.1" />
 			<inertia
 			  ixx="0.4708"
@@ -58,5 +58,5 @@
 		<inertial>
 		    	<origin rpy="0 0 ${Angle_Sail2}" xyz="-0.3 0 0.4"/>
-			<mass value="1" />
+			<mass value="0.1" />
 			<inertia
 			  ixx="0.4708"
@@ -93,5 +93,5 @@
     <link name="keel">
 	<inertial>
-		<mass value="30" />
+		<mass value="0.3" />
 		<inertia
 		  ixx="0.4708"
@@ -104,5 +104,5 @@
 	<collision name="collision">
 		<geometry>
-			<box size="0.25 0.02 0.5" />
+			<box size="0.045 0.02 0.315" />
 		</geometry>
 		<origin rpy="0 0 0" xyz="0 0 0"/>
@@ -110,5 +110,5 @@
 	<visual name="visual">
 		<geometry>
-			<mesh filename="package://usv_sim/meshes/simpleHull3/box.dae" scale="0.25 0.02 0.5"/>
+			<mesh filename="package://usv_sim/meshes/simpleHull3/box.dae" scale="0.045 0.02 0.315"/>
 		</geometry>
 		<origin rpy="0 0 0" xyz="0 0 0"/>
@@ -118,5 +118,37 @@
         <parent link="base_link"/>
         <child link="keel"/>
-        <origin rpy="0 0 0" xyz="0 0 -0.12"/>
+        <origin rpy="0 0 0" xyz="0 0 -0.18"/>
+        <dynamics damping="1.0"/>
+        <axis xyz="0 0 1"/>
+        <limit effort="30" velocity="5" lower="0" upper="0" />
+    </joint>
+    <link name="subkeel">
+	<inertial>
+		<mass value="2.2" />
+		<inertia
+		  ixx="0.4708"
+		  ixy="0.0"
+		  iyy="0.5208"
+		  ixz="0.0"
+		  iyz="0.0"
+		  izz="0.0508"/>
+	</inertial>
+	<collision name="collision">
+		<geometry>
+			<mesh filename="package://usv_sim/meshes/simpleHull3/Torpedo_keel.dae" scale="0.03333 0.0262 0.03333"/>
+		</geometry>
+		<origin rpy="0 0 1.57" xyz="0 0 0"/>
+	</collision>
+	<visual name="visual">
+		<geometry>
+			<mesh filename="package://usv_sim/meshes/simpleHull3/Torpedo_keel.dae" scale="0.03333 0.0262 0.03333"/>
+		</geometry>
+		<origin rpy="0 0 1.57" xyz="0 0 0"/>
+	</visual>
+</link>
+    <joint name="subkeel_joint" type="revolute">
+        <parent link="keel"/>
+        <child link="subkeel"/>
+        <origin rpy="0 0 0" xyz="0.1 0 -0.16"/>
         <dynamics damping="1.0"/>
         <axis xyz="0 0 1"/>
@@ -138,5 +170,5 @@
 		<cp>0 0 0</cp>
 		<joint_name>sail_joint</joint_name>
-		<area>1.44</area>
+		<area>0.275</area>
 		<fluid_density>1.2041</fluid_density>
 		<forward>-1 0 0</forward>
@@ -157,5 +189,5 @@
 		<cp>0 0 0</cp>
 		<joint_name>sail_joint_2</joint_name>
-		<area>1.44</area>
+		<area>0.225</area>
 		<fluid_density>1.2041</fluid_density>
 		<forward>-1 0 0</forward>
