Commit message: 23 feb

File: Versions/Actual_version/Model/boat_subdivided4.xacro (robot description, xacro)
@@ -3,15 +3,15 @@
     <xacro:property name="PI" value="3.1415926535897931"/>
     <!-- Body properties -->
-    <xacro:property name="front_body_mass" value="5"/>
-    <xacro:property name="back_body_mass" value="5"/>
-    <xacro:property name="middle_body_mass" value="5"/>
-    <xacro:property name="rear_body_mass" value="5"/>
-    <xacro:property name="front_body_mass" value="2"/>
-    <xacro:property name="back_water_displaced_mass" value="26"/>
-    <xacro:property name="middle_water_displaced_mass" value="26"/>
-    <xacro:property name="front_water_displaced_mass" value="15"/>
-    <xacro:property name="scalex" value=".3"/>
-    <xacro:property name="scaley" value=".2"/>
-    <xacro:property name="scalez" value=".3"/>
+    <xacro:property name="front_body_mass" value="0.3"/>
+    <xacro:property name="back_body_mass" value="0.3"/>
+    <xacro:property name="middle_body_mass" value="0.3"/>
+    <xacro:property name="rear_body_mass" value="0.3"/>
+    <xacro:property name="front_body_mass" value="0.3"/>
+    <xacro:property name="back_water_displaced_mass" value="40"/>
+    <xacro:property name="middle_water_displaced_mass" value="40"/>
+    <xacro:property name="front_water_displaced_mass" value="25"/>
+    <xacro:property name="scalex" value=".193"/>
+    <xacro:property name="scaley" value=".117"/>
+    <xacro:property name="scalez" value=".1"/>
     <xacro:property name="bl1" value=".1" />
     <xacro:property name="bl2" value=".1" />
@@ -370,5 +370,5 @@
             <parent link="back_r_link"/>
             <child link="rudder"/>
-            <origin rpy="0 0 0" xyz="${-1.4*scalex} ${0.39*scaley} ${-0.5*scalez}"/>
+            <origin rpy="0 0 0" xyz="-0.25 0.04 -0.10"/>
             <dynamics damping="1.0"/>
             <axis xyz="0 0 1"/>

File: Versions/Actual_version/Model/sailboat.xacro (robot description, xacro)
@@ -5,13 +5,23 @@
     <xacro:property name="windType" value="$(arg windType)" />
     <xacro:property name="waterType" value="$(arg waterType)" />
+    <xacro:property name="scale_V1X" value="0.325"/>
+    <xacro:property name="scale_V1Y" value="0.325"/>
+    <xacro:property name="scale_V1Z" value="0.637"/>
+    <xacro:property name="scale_V2X" value="0.335"/>
+    <xacro:property name="scale_V2Y" value="0.335"/>
+    <xacro:property name="scale_V2Z" value="0.51"/>
     <xacro:property name="Angle_Sail2" value="3.14"/>
+    <xacro:property name="SailXo" value="0.04"/>
+    <xacro:property name="SailYo" value="0"/>
+    <xacro:property name="SailZo" value="-0.041"/>
     <xacro:property name="windType" value="global"/>
     <xacro:include filename="$(find usv_sim)/xacro/boat_subdivided4.xacro" />
     <xacro:rudder_xacro/>
     <!-- Defining sail model -->
+     <!-- Vela1 -->
     <link name="sail">
 		<inertial>
 		    	<origin rpy="0 0 0" xyz="-0.3 0 0.4"/>
-			<mass value="1" />
+			<mass value="0.1" />
 			<inertia
 			  ixx="0.4708"
@@ -24,5 +34,5 @@
 	    <collision name="collision">
             <geometry>
-              <mesh filename="package://usv_sim/meshes/simpleHull3/sail.dae" scale="0.5 0.5 1"/>
+              <mesh filename="package://usv_sim/meshes/simpleHull3/sail.dae" scale="${scale_V1X} ${scale_V1Y} ${scale_V1Z}"/>
             </geometry>
             <origin rpy="0 0 0" xyz="0 0 0"/>
@@ -30,5 +40,5 @@
 	    <visual name="visual">
             <geometry>
-              <mesh filename="package://usv_sim/meshes/simpleHull3/sail.dae" scale="0.5 0.5 1"/>
+              <mesh filename="package://usv_sim/meshes/simpleHull3/sail.dae" scale="${scale_V1X} ${scale_V1Y} ${scale_V1Z}"/>
             </geometry>
             <origin rpy="0 0 0" xyz="0 0 0"/>
@@ -38,13 +48,15 @@
         <parent link="base_link"/>
         <child link="sail"/>
-        <origin rpy="0 0 0" xyz="0.2 0 -0.07"/>
-        <dynamics damping="1.0"/>
-        <axis xyz="0 0 1"/>
-        <limit effort="100" velocity="70" lower="-3.14" upper="3.14" />
-    </joint>
+        <origin rpy="0 0 0" xyz="${SailXo} ${SailYo} ${SailZo}"/>
+        <dynamics damping="1.0"/>
+        <axis xyz="0 0 1"/>
+        <limit effort="100" velocity="70" lower="-${PI}" upper="${PI}" />
+    </joint>
+<!-- ******************************************************************************************* -->
+ <!-- Vela2 -->
     <link name="sail_2">
 		<inertial>
 		    	<origin rpy="0 0 ${Angle_Sail2}" xyz="-0.3 0 0.4"/>
-			<mass value="1" />
+			<mass value="0.1" />
 			<inertia
 			  ixx="0.4708"
@@ -57,5 +69,5 @@
 	    <collision name="collision">
             <geometry>
-              <mesh filename="package://usv_sim/meshes/simpleHull3/sail.dae" scale="0.5 0.5 0.8"/>
+              <mesh filename="package://usv_sim/meshes/simpleHull3/sail.dae" scale="${scale_V2X} ${scale_V2Y} ${scale_V2Z}"/>
             </geometry>
             <origin rpy="0 0 ${Angle_Sail2}" xyz="0 0 0"/>
@@ -63,5 +75,5 @@
 	    <visual name="visual">
             <geometry>
-              <mesh filename="package://usv_sim/meshes/simpleHull3/sail.dae" scale="0.5 0.5 0.8"/>
+              <mesh filename="package://usv_sim/meshes/simpleHull3/sail.dae" scale="${scale_V2X} ${scale_V2Y} ${scale_V2Z}"/>
             </geometry>
             <origin rpy="0 0 ${Angle_Sail2}" xyz="0 0 0"/>
@@ -71,13 +83,15 @@
         <parent link="base_link"/>
         <child link="sail_2"/>
-        <origin rpy="0 0 0" xyz="0.2 0 0"/>
+        <origin rpy="0 0 0" xyz="${SailXo} ${SailYo} ${SailZo+0.044}"/>
 <!-- valores originales 0.2, 0 ,0.1-->
         <dynamics damping="1.0"/>
         <axis xyz="0 0 1"/>
-        <limit effort="100" velocity="70" lower="-3.14" upper="3.14" />
-    </joint>
+        <limit effort="100" velocity="70" lower="-${PI}" upper="${PI}" />
+    </joint>
+<!-- ******************************************************************************************* -->
+<!-- Quilla -->
     <link name="keel">
 	<inertial>
-		<mass value="30" />
+		<mass value="0.3" />
 		<inertia
 		  ixx="0.4708"
@@ -90,5 +104,5 @@
 	<collision name="collision">
 		<geometry>
-			<box size="0.25 0.02 0.5" />
+			<box size="0.045 0.02 0.315" />
 		</geometry>
 		<origin rpy="0 0 0" xyz="0 0 0"/>
@@ -96,5 +110,5 @@
 	<visual name="visual">
 		<geometry>
-			<mesh filename="package://usv_sim/meshes/simpleHull3/box.dae" scale="0.25 0.02 0.5"/>
+			<mesh filename="package://usv_sim/meshes/simpleHull3/box.dae" scale="0.045 0.02 0.315"/>
 		</geometry>
 		<origin rpy="0 0 0" xyz="0 0 0"/>
@@ -104,9 +118,42 @@
         <parent link="base_link"/>
         <child link="keel"/>
-        <origin rpy="0 0 0" xyz="0 0 -0.35"/>
+        <origin rpy="0 0 0" xyz="0 0 -0.18"/>
         <dynamics damping="1.0"/>
         <axis xyz="0 0 1"/>
         <limit effort="30" velocity="5" lower="0" upper="0" />
     </joint>
+    <link name="subkeel">
+	<inertial>
+		<mass value="2.2" />
+		<inertia
+		  ixx="0.4708"
+		  ixy="0.0"
+		  iyy="0.5208"
+		  ixz="0.0"
+		  iyz="0.0"
+		  izz="0.0508"/>
+	</inertial>
+	<collision name="collision">
+		<geometry>
+			<mesh filename="package://usv_sim/meshes/simpleHull3/Torpedo_keel.dae" scale="0.03333 0.0262 0.03333"/>
+		</geometry>
+		<origin rpy="0 0 1.57" xyz="0 0 0"/>
+	</collision>
+	<visual name="visual">
+		<geometry>
+			<mesh filename="package://usv_sim/meshes/simpleHull3/Torpedo_keel.dae" scale="0.03333 0.0262 0.03333"/>
+		</geometry>
+		<origin rpy="0 0 1.57" xyz="0 0 0"/>
+	</visual>
+</link>
+    <joint name="subkeel_joint" type="revolute">
+        <parent link="keel"/>
+        <child link="subkeel"/>
+        <origin rpy="0 0 0" xyz="0.1 0 -0.16"/>
+        <dynamics damping="1.0"/>
+        <axis xyz="0 0 1"/>
+        <limit effort="30" velocity="5" lower="0" upper="0" />
+    </joint>
+<!-- ******************************************************************************************* -->
     <!-- Plugin list -->
   <gazebo>
@@ -123,5 +170,5 @@
 		<cp>0 0 0</cp>
 		<joint_name>sail_joint</joint_name>
-		<area>1.44</area>
+		<area>0.275</area>
 		<fluid_density>1.2041</fluid_density>
 		<forward>-1 0 0</forward>
